File: rocket-mega-shield.brd (EAGLE design)
At the start: 101.6 x 53.6 mm, 66 parts, among them J1 ExtBatt, J2 Mega R3, J3 XBEE, J4 MICROSD, J5 U.FL, J6 1X6TERMINALBLOCK, Q1 SI7112DN, Q2 BSS138, Q3 BSS138, Q4 SI7112DN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

Commit message: more cleanup on the 2.1 board
Parts:
- Q1, Q4, Q5, Q6, Q7: device SparkFun-DiscreteSemi:POWERPAK1212-8 -> zortness:POWERPAK1212-8
- U1: device kurt:DPAK -> zortness:DPAK
- U3: device adafruit:FGPMMOPA6H -> zortness:FGPMMOPA6H
- moved C17 5.58 mm to (81.4, 9.05)
- moved C19 5.01 mm to (87.3, 9.05), turned to 0 degrees
- moved C18 4.47 mm to (75.6, 9.05)
- moved C21 4.44 mm to (71.1, 12.1)
- moved U7 3.17 mm to (80.0, 13.3)
- moved U1 0.63 mm to (31.1, 12.1)
Connections:
- net MEGAA10: now also C19.1, U7.5; no longer C18.1, U7.16
- net MEGAA8: now also C18.1, U7.16; no longer C19.1, U7.5
Routing:
- net MEGAA8: track 29.5 -> 11.7 mm
- net MEGAA9: track 19.0 -> 11.0 mm
- net MEGAA10: track 10.9 -> 16.7 mm
- net VIN: track 69.7 -> 67.2 mm
- net VCC3: track 327.7 -> 328.9 mm
