File: rocket-mega-shield.sch (EAGLE design)
At the start: 64 parts, among them J1 ExtBatt, J2 MICROSD, J3 Mega R3, J4 1X6TERMINALBLOCK, J5 XBEE, J6 U.FL, Q1 BSS138, Q2 BSS138, Q3 SI7112DN, Q4 SI7112DN, Q5 SI7112DN, Q6 SI7112DN, Q7 BSS138, U1 BMP180, U2 FGPMMOPA6H, U3 NCP1117DT33G, U6 LSM303DLHCTR, U7 L3GD20TR, U8 ADXL377, U9 M74HC4050M

Commit message: routing and visual cleanup
Parts:
- removed C22, C23: 0.1uF, adafruit:C-USC1206
- removed U8: ADXL377, zortness:ADXL377
- removed U9: M74HC4050M, SparkFun-DigitalIC:HEX_CONVERTER
- added C5: 10uF, adafruit:C-USC1206
- added C6: 100uF16V, adafruit:C-USC1210
- added U4: BMP180, zortness:BMP180
- added U5: LSM303DLHCTR, kurt:LSM303DLHC
- C1: value 100uF -> 10uF
- C10: value 10uF -> 0.22uF
- C12: value 0.22uF -> 4.7uF
- C13: value 0.01uF -> 10uF
- C14, C21: value 10uF -> 0.1uF
- C15: value 0.1uF -> 10uF
- C16: value 1uF -> 0.1uF
- C2: value 100uF16V -> 0.1uF; device adafruit:C-USC1210 -> adafruit:C-USC1206
- C3: value 10uF -> 100uF
- C8: value 0.1uF -> 1uF
- C9: value 4.7uF -> 0.01uF
- D10: value 13 - red -> Pyro4 - red
- D2: value PWR - green -> 13 - red
- D3: value SDAct - orange -> Fix - blue
- D5: value Fix - blue -> SDAct - orange
- D6: value Pyro1 - red -> PWR - green
- D7: value Pyro2 - red -> Pyro1 - red
- D8: value Pyro3 - red -> Pyro2 - red
- D9: value Pyro4 - red -> Pyro3 - red
- J2: value MICROSD -> Mega R3; device zortness:MICROSD -> zortness:ARDUINO-MEGAFULL
- J3: value Mega R3 -> XBEE; device kurt:ARDUINO-MEGAFULL -> adafruit:XBEE
- J4: value 1X6TERMINALBLOCK -> MICROSD; device zortness:1X6TERMINALBLOCK -> zortness:MICROSD
- J5: value XBEE -> U.FL; device adafruit:XBEE -> SparkFun-Connectors:U.FL
- J6: value U.FL -> 1X6TERMINALBLOCK; device SparkFun-Connectors:U.FL -> zortness:1X6TERMINALBLOCK
- Q3: value SI7112DN -> BSS138; device SparkFun-DiscreteSemi:MOSFET-NCHANNELSI7820DN -> kurt:BSS138
- Q7: value BSS138 -> SI7112DN; device kurt:BSS138 -> SparkFun-DiscreteSemi:MOSFET-NCHANNELSI7820DN
- R1, RA3: value 620k -> 110k
- R2, RA4: value 110k -> 620k
- R3: value 10k -> 330
- R4: value 330 -> 10k
- S1: value AYZ0202 -> KMR2; device SparkFun-Electromechanical:AYZ0202 -> zortness:TAC_SWITCHKMR2
- S2: value KMR2 -> AYZ0202; device zortness:TAC_SWITCHKMR2 -> SparkFun-Electromechanical:AYZ0202
- U1: value BMP180 -> NCP1117DT33G; device zortness:BMP180 -> kurt:NCP1117DT33G
- U2: value FGPMMOPA6H -> M74HC4050M; device adafruit:GPS_FGPMMOPA6H -> SparkFun-DigitalIC:HEX_CONVERTER
- U3: value NCP1117DT33G -> FGPMMOPA6H; device kurt:NCP1117DT33G -> adafruit:GPS_FGPMMOPA6H
- U6: value LSM303DLHCTR -> L3GD20TR; device kurt:LSM303DLHC -> kurt:L3GD20
- U7: value L3GD20TR -> ADXL377; device kurt:L3GD20 -> zortness:ADXL377
- renumbered C26 to C18
Connections:
- net BATT+: now also J6.1, J6.2; no longer J4.1, J4.2
- net GND: now also C12.2, C5.2, C6.2, J2.GND@0, J2.GND@1, J2.GND@2, J2.GND@3, J2.GND@4, J3.GND, J4.CARD_DETECT, J4.CARD_DETECT1, J4.GND, J4.GND1, J4.VSS, J5.GND@0, J5.GND@1, Q1.SRC, Q7.S, R1.1, R4.2, RA2.A2, RA2.B2, RA2.C2, RA2.D2, RA3.A1, RA3.B1, RA3.C1, RA3.D1, S1.3, S1.4, U2.GND, U3.GND@1, U3.GND@2, U3.GND@3, U3.GND@4, U4.GND, U5.GND@1, U5.GND@2, U5.GND@3, U6.GND@10, U6.GND@11, U6.GND@12, U6.GND@13, U6.GND@8, U6.GND@9, U7.GND@1, U7.GND@2; no longer C10.2, C22.2, C23.2, J2.CARD_DETECT, J2.CARD_DETECT1, J2.GND, J2.GND1, J2.VSS, J3.GND@0, J3.GND@1, J3.GND@2, J3.GND@3, J3.GND@4, J5.GND, J6.GND@0, J6.GND@1, Q3.S, Q7.SRC, R2.1, R3.2, RA4.A1, RA4.B1, RA4.C1, RA4.D1, RA6.A2, RA6.B2, RA6.C2, RA6.D2, S2.3, S2.4, U2.GND@1, U2.GND@2, U2.GND@3, U2.GND@4, U3.GND, U6.GND@1, U6.GND@2, U6.GND@3, U7.GND@10, U7.GND@11, U7.GND@12, U7.GND@13, U7.GND@8, U7.GND@9, U8.GND@1, U8.GND@2, U9.GND
- net GPSFIX: now also U3.3D-FIX; no longer U2.3D-FIX
- net IOREF: now also J2.IOREF, RA6.A1, RA6.B1; no longer J3.IOREF, RA2.A1, RA2.B1
- net MEGA5V: now also J2.5V@0; no longer J3.5V@0
- net MEGA8: now also J2.8, Q1.GTE, R4.1; no longer J3.8, Q7.GTE, R3.1
- net MEGAA0: now also J2.A0(RX0); no longer J3.A0(RX0)
- net MEGAA1: now also J2.A1(TX0); no longer J3.A1(TX0)
- net MEGAA10: now also J2.A10, U7.Z; no longer J3.A10, U8.Z
- net MEGAA11: now also J2.A11, RA3.D2, RA4.D1; no longer J3.A11, RA3.D1, RA4.D2
- net MEGAA12: now also J2.A12, RA3.C2, RA4.C1; no longer J3.A12, RA3.C1, RA4.C2
- net MEGAA13: now also J2.A13, RA3.B2, RA4.B1; no longer J3.A13, RA3.B1, RA4.B2
- net MEGAA14: now also J2.A14, RA3.A2, RA4.A1; no longer J3.A14, RA3.A1, RA4.A2
- net MEGAA15: now also J2.A15, R1.2, R2.1; no longer J3.A15, R1.1, R2.2
- net MEGAA2: now also J2.A2; no longer J3.A2
- net MEGAA3: now also J2.A3; no longer J3.A3
- net MEGAA4: now also J2.A4; no longer J3.A4
- net MEGAA5: now also J2.A5; no longer J3.A5
- net MEGAA6: now also J2.A6; no longer J3.A6
- net MEGAA7: now also J2.A7; no longer J3.A7
- net MEGAA8: now also J2.A8, U7.X; no longer J3.A8, U8.X
- net MEGAA9: now also C17.1, J2.A9, U7.Y; no longer C20.1, J3.A9, U8.Y
- net MEGAMISO: now also J2.50, J4.DATA_OUT; no longer J2.DATA_OUT, J3.50
- net MEGAMOSI: now also J2.51, U2.4A; no longer J3.51, U9.4A
- net MEGARX0: now also J2.0(RX0), S2.6; no longer J3.0(RX0), S1.6
- net MEGARX1: now also J2.19(RX1), S2.4; no longer J3.19(RX1), S1.4
- net MEGARX2: now also J2.17(RX2), U3.TX; no longer J3.17(RX2), U2.TX
- net MEGASCL: now also J2.21(SCL), Q3.DRN, RA6.B2; no longer J3.21(SCL), Q2.DRN, RA2.B2
- net MEGASCLK: now also J2.52, U2.5A; no longer J3.52, U9.5A
- net MEGASDA: now also J2.20(SDA), Q2.DRN, RA6.A2; no longer J3.20(SDA), Q1.DRN, RA2.A2
- net MEGASDCS: now also J2.48, U2.6A; no longer J3.48, U9.6A
- net MEGATX0: now also J2.1(TX0), U2.1A; no longer J3.1(TX0), U9.1A
- net MEGATX1: now also J2.18(TX1), U2.2A; no longer J3.18(TX1), U9.2A
- net MEGATX2: now also J2.16(TX2), U2.3A; no longer J3.16(TX2), U9.3A
- net MOSI: now also J4.DATA_IN, U2.4Y; no longer J2.DATA_IN, U9.4Y
- net N$1: now also D6.A; no longer D2.A
- net N$10: now also J5.SIGNAL, U3.EX_ANT; no longer J6.SIGNAL, U2.EX_ANT
- net N$12: now also D3.A; no longer D5.A
- net N$13: now also Q1.DRN; no longer Q7.DRN
- net N$14: now also D2.A, R3.2; no longer D10.A, R4.2
- net N$16: now also D10.A; no longer D9.A
- net N$17: now also D9.A; no longer D8.A
- net N$18: now also D8.A; no longer D7.A
- net N$19: now also D7.A; no longer D6.A
- net N$2: now also D5.A; no longer D3.A
- net N$21: now also J3.DOUT, S2.5; no longer J5.DOUT, S1.5
- net N$22: now also J3.DIN, S2.2; no longer J5.DIN, S1.2
- net N$24: now also J6.6, Q5.D, RA4.A2; no longer J4.6, Q6.D, RA3.A2
- net N$25: now also J6.5, Q6.D, RA4.B2; no longer J4.5, Q5.D, RA3.B2
- net N$3: now also J6.3, Q7.D, RA4.D2; no longer J4.3, Q3.D, RA3.D2
- net N$4: now also J6.4, RA4.C2; no longer J4.4, RA3.C2
- net N$5: now also C10.2, U5.SETP_C2; no longer C12.2, U6.SETP_C2
- net N$6: now also C10.1, U5.SETC_C2; no longer C12.1, U6.SETC_C2
- net N$7: now also C12.1, U5.C1; no longer C9.1, U6.C1
- net N$8: now also C20.1, U6.GND@14; no longer C13.1, U7.GND@14
- net N$9: now also J2.13, R3.1; no longer J3.13, R4.1
- net PYRO1: now also J2.42, Q7.G, RA2.A1; no longer J3.42, Q3.G, RA6.A1
- net PYRO2: now also J2.43, RA2.B1; no longer J3.43, RA6.B1
- net PYRO3: now also J2.44, Q6.G, RA2.C1; no longer J3.44, Q5.G, RA6.C1
- net PYRO4: now also J2.45, Q5.G, RA2.D1; no longer J3.45, Q6.G, RA6.D1
- net RESET: now also J2.RESET, S1.1, S1.2; no longer J3.RESET, S2.1, S2.2
- net SCL: now also Q3.SRC, RA6.C2, U4.SCL, U5.SCL, U6.SCL/SCP; no longer Q2.SRC, RA2.C2, U1.SCL, U6.SCL, U7.SCL/SCP
- net SCLK: now also J4.SCLK, U2.5Y; no longer J2.SCLK, U9.5Y
- net SDA: now also Q2.SRC, RA6.D2, U4.SDA, U5.SDA, U6.SDA/SDI; no longer Q1.SRC, RA2.D2, U1.SDA, U6.SDA, U7.SDA/SDI
- net SDCS: now also J4.CS, U2.6Y; no longer J2.CS, U9.6Y
- net TX0: now also S2.3, U2.1Y; no longer S1.3, U9.1Y
- net TX1: now also S2.1, U2.2Y; no longer S1.1, U9.2Y
- net TX2: now also U2.3Y, U3.RX; no longer U2.RX, U9.3Y
- net VCC3: now also C13.1, C2.1, C5.1, C9.1, J3.VCC, J4.VDD, Q3.GTE, RA6.C1, RA6.D1, U1.OUT, U3.VCC, U4.VDD, U4.VDDIO, U5.VDD, U5.VDD_IO, U6.VDD@1, U6.VDD@2, U7.VS@1, U7.VS@2; no longer C10.1, C17.1, C22.1, C23.1, J2.VDD, J5.VCC, Q1.GTE, RA2.C1, RA2.D1, U1.VDD, U1.VDDIO, U3.OUT, U6.VDD, U7.VDD@1, U7.VDD@2, U7.VDD_IO, U8.VS@1, U8.VS@2, U9.VCC
- net VIN: now also C6.1, J2.VIN, R2.2, U1.IN; no longer C2.1, J3.VIN, R1.2, U3.IN
- net XRSSI: now also J3.PWM0/RSSI; no longer J5.PWM0/RSSI
Other:
- moved on the sheet: C1, C10, C11, C12, C13, C14, C15, C16, C17, C2, C20, C21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

Commit message: changed out mosfet on speaker for higher amperage, more cleanup
Parts:
- added LOGO1: OSHW-LOGOM, SparkFun-Aesthetics:OSHW-LOGOM
- Q1: value BSS138 -> SI7112DN; device kurt:BSS138 -> SparkFun-DiscreteSemi:MOSFET-NCHANNELSI7820DN
- R1, RA3: value 110k -> 100k
Connections:
- net GND: now also Q1.S; no longer Q1.SRC
- net MEGA8: now also Q1.G; no longer Q1.GTE
- net N$13: now also Q1.D; no longer Q1.DRN
Changed lines of the file:
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@@
 <setting verticaltext="up"/>
 </settings>
-<grid distance="0.1" unitdist="inch" unit="inch" style="lines" multiple="1" display="no" altdistance="0.01" altunitdist="inch" altunit="inch"/>
+<grid distance="0.05" unitdist="inch" unit="inch" style="lines" multiple="1" display="no" altdistance="0.025" altunitdist="inch" altunit="inch"/>
 <layers>
 <layer number="1" name="Top" color="4" fill="1" visible="no" active="no"/>
@@
 <layer number="199" name="Contour" color="7" fill="1" visible="yes" active="yes"/>
 <layer number="200" name="200bmp" color="1" fill="10" visible="yes" active="yes"/>
-<layer number="201" name="201bmp" color="2" fill="1" visible="no" active="no"/>
+<layer number="201" name="201bmp" color="2" fill="10" visible="yes" active="yes"/>
 <layer number="202" name="202bmp" color="3" fill="1" visible="no" active="no"/>
 <layer number="203" name="203bmp" color="4" fill="10" visible="yes" active="yes"/>
@@
 <part name="RA6" library="zortness" deviceset="RESISTOR_CRA06S08" device="" value="10k"/>
 <part name="RA4" library="zortness" deviceset="RESISTOR_CRA06S08" device="" value="620k"/>
-<part name="RA3" library="zortness" deviceset="RESISTOR_CRA06S08" device="" value="110k"/>
+<part name="RA3" library="zortness" deviceset="RESISTOR_CRA06S08" device="" value="100k"/>
 <part name="GND35" library="supply1" deviceset="GND" device=""/>
 <part name="RA5" library="zortness" deviceset="RESISTOR_CRA06S08" device="" value="330"/>
@@
 <part name="GND41" library="supply1" deviceset="GND" device=""/>
 <part name="R2" library="adafruit" deviceset="R-US_" device="R1206" value="620k"/>
-<part name="R1" library="adafruit" deviceset="R-US_" device="R1206" value="110k"/>
+<part name="R1" library="adafruit" deviceset="R-US_" device="R1206" value="100k"/>
 <part name="GND13" library="supply1" deviceset="GND" device=""/>
 <part name="U4" library="zortness" deviceset="BMP180" device="" value="BMP180"/>
 <part name="S1" library="zortness" deviceset="TAC_SWITCH" device="KMR2" value="KMR2"/>
-<part name="Q1" library="kurt" deviceset="BSS138" device="" value="BSS138"/>
 <part name="R4" library="adafruit" deviceset="R-US_" device="R1206" value="10k"/>
 <part name="GND14" library="supply1" deviceset="GND" device=""/>
@@
 <part name="R3" library="adafruit" deviceset="R-US_" device="R1206" value="330"/>
 <part name="GND20" library="supply1" deviceset="GND" device=""/>
+<part name="LOGO1" library="SparkFun-Aesthetics" deviceset="OSHW-LOGO" device="M"/>
+<part name="Q1" library="SparkFun-DiscreteSemi" deviceset="MOSFET-NCHANNEL" device="SI7820DN" value="SI7112DN"/>
 </parts>
 <sheets>
@@
 <instance part="U4" gate="G$1" x="137.16" y="30.48"/>
 <instance part="S1" gate="S" x="-152.4" y="43.18" rot="R90"/>
-<instance part="Q1" gate="G$1" x="55.88" y="10.16" rot="R180"/>
 <instance part="R4" gate="G$1" x="76.2" y="12.7" rot="R90"/>
 <instance part="GND14" gate="1" x="76.2" y="25.4" rot="R180"/>
@@
 <instance part="R3" gate="G$1" x="-78.74" y="55.88"/>
 <instance part="GND20" gate="1" x="-66.04" y="53.34" rot="MR0"/>
+<instance part="LOGO1" gate="G$1" x="-60.96" y="127"/>
+<instance part="Q1" gate="G$1" x="59.69" y="15.24" rot="R90"/>
 </instances>
 <busses>
@@
 <pinref part="GND14" gate="1" pin="GND"/>
 <wire x1="76.2" y1="17.78" x2="76.2" y2="20.32" width="0.1524" layer="91"/>
-<pinref part="Q1" gate="G$1" pin="SRC"/>
 <wire x1="76.2" y1="20.32" x2="76.2" y2="22.86" width="0.1524" layer="91"/>
-<wire x1="66.04" y1="12.7" x2="68.58" y2="12.7" width="0.1524" layer="91"/>
-<wire x1="68.58" y1="12.7" x2="68.58" y2="20.32" width="0.1524" layer="91"/>
+<wire x1="64.77" y1="15.24" x2="68.58" y2="15.24" width="0.1524" layer="91"/>
+<wire x1="68.58" y1="15.24" x2="68.58" y2="20.32" width="0.1524" layer="91"/>
 <wire x1="68.58" y1="20.32" x2="76.2" y2="20.32" width="0.1524" layer="91"/>
 <junction x="76.2" y="20.32"/>
+<pinref part="Q1" gate="G$1" pin="S"/>
 </segment>
 <segment>
@@
 <net name="N$13" class="0">
 <segment>
-<pinref part="Q1" gate="G$1" pin="DRN"/>
 <wire x1="50.8" y1="10.16" x2="45.72" y2="10.16" width="0.1524" layer="91"/>
 <pinref part="SG1" gate="G$1" pin="1"/>
+<wire x1="50.8" y1="10.16" x2="50.8" y2="15.24" width="0.1524" layer="91"/>
+<pinref part="Q1" gate="G$1" pin="D"/>
+<wire x1="50.8" y1="15.24" x2="54.61" y2="15.24" width="0.1524" layer="91"/>
 </segment>
 </net>
@@
 </segment>
 <segment>
-<pinref part="Q1" gate="G$1" pin="GTE"/>
-<wire x1="66.04" y1="7.62" x2="76.2" y2="7.62" width="0.1524" layer="91"/>
 <label x="78.74" y="7.62" size="1.778" layer="95"/>
 <pinref part="R4" gate="G$1" pin="1"/>
 <wire x1="76.2" y1="7.62" x2="86.36" y2="7.62" width="0.1524" layer="91"/>
+<pinref part="Q1" gate="G$1" pin="G"/>
+<wire x1="76.2" y1="7.62" x2="59.69" y2="7.62" width="0.1524" layer="91"/>
 <junction x="76.2" y="7.62"/>
 </segment>

Commit message: changed mosfet for speaker, added osaerospace logo
Parts:
- added U$1: OSAEROSPACEVECTOR, zortness:OSAEROSPACEVECTOR
Other:
- note added: "Designed by Kurtis Kopf"
- note added: "OpenSourceAerospace.com"
Changed lines of the file:
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@@
 <part name="LOGO1" library="SparkFun-Aesthetics" deviceset="OSHW-LOGO" device="M"/>
 <part name="Q1" library="SparkFun-DiscreteSemi" deviceset="MOSFET-NCHANNEL" device="SI7820DN" value="SI7112DN"/>
+<part name="U$1" library="zortness" deviceset="OSAEROSPACE" device="VECTOR"/>
 </parts>
 <sheets>
@@
 <wire x1="88.9" y1="0" x2="88.9" y2="35.56" width="0.1524" layer="97"/>
 <wire x1="88.9" y1="35.56" x2="33.02" y2="35.56" width="0.1524" layer="97"/>
+<text x="-140.97" y="121.92" size="1.778" layer="97" font="vector">Designed by Kurtis Kopf</text>
+<text x="-140.97" y="119.38" size="1.778" layer="97" font="vector">OpenSourceAerospace.com</text>
 </plain>
 <instances>
@@
 <instance part="LOGO1" gate="G$1" x="-60.96" y="127"/>
 <instance part="Q1" gate="G$1" x="59.69" y="15.24" rot="R90"/>
+<instance part="U$1" gate="G$1" x="-34.29" y="125.73"/>
 </instances>
 <busses>

Commit message: changed out xbee to clean up screen printing lines, trimmed working window down to actual board size
Parts:
- J3: device adafruit:XBEE -> zortness:XBEE
Changed lines of the file:
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@@
 </classes>
 <parts>
-<part name="J3" library="adafruit" deviceset="XBEE" device=""/>
+<part name="J3" library="zortness" deviceset="XBEE" device=""/>
 <part name="J4" library="zortness" deviceset="MICROSD" device=""/>
 <part name="U3" library="adafruit" deviceset="GPS_FGPMMOPA6H" device="" value="FGPMMOPA6H"/>
